File: schematic/schematic.sch (KiCad schematic (older format))
At the start: 56 parts

Commit message: update main schematic
Parts:
- removed C?: 4.7uF, symbol Device:C_Small
- removed C? (x3): 2.2uF, symbol Device:C_Small
- removed C?: 100nF, symbol Device:C_Small
- added C? (x4): 2.2uF, symbol Device:CP1_Small
- added C?: 10nF, symbol Device:C_Small
- added C?: 0.1uF, symbol Device:C_Small
- added C? (x3): 100nF, symbol Device:C_Small
- added F?: 500mA, symbol Device:Polyfuse_Small
- added J?: ICSP, symbol Connector_Generic:Conn_02x03_Odd_Even
- added L?: 10uH, symbol Device:L_Small
- added R?: 8.2k, symbol Device:R_Small
- added R?: 12k, symbol Device:R_Small
- added R?: 10k, symbol Device:R_Small
- added SW?: SW_RESET, symbol Switch:SW_Push
- C?: value 47pF -> 22pF
- R?: value 6k -> 5.6k
- R?: value 75k -> 150k
- R? (x2): value 75k -> 100k
- R?: value 6k -> 51k
Connections:
- net labels added: A0, A1, A2, MISO, MOSI, RESET, RX, SCK, TX, ~DTR
- wire segments 180 -> 214
- no-connect marks 8 -> 17
Other:
- moved on the sheet: C?, D?, R?, U?, U?A, U?B, U?C, U?D, U?E, Y?

Commit message: initial processing board
Parts:
- C?: value 0.1uF -> 100nF
Changed lines of the file:
@@
 P 4750 950
 F 0 "C?" H 4842 996 50  0000 L CNN
-F 1 "0.1uF" H 4842 905 50  0000 L CNN
+F 1 "100nF" H 4842 905 50  0000 L CNN
 F 2 "" H 4750 950 50  0001 C CNN
 F 3 "~" H 4750 950 50  0001 C CNN

Commit message: audio system approved
Parts:
- removed C? (x4): C_Small, symbol Device:C_Small
- removed C?: 2.2uF, symbol Device:CP1_Small
- removed MK? (x2): Microphone, symbol Device:Microphone
- removed R? (x6): R_Small, symbol Device:R_Small
- removed R? (x2): 100k, symbol Device:R_Small
- removed U? (x5): Opamp_Quad_Generic, symbol Device:Opamp_Quad_Generic
- added C? (x4): 4.7nF, symbol Device:C_Small
- added C? (x2): 22pF, symbol Device:C_Small
- added C? (x7): 2.2uF, symbol Device:CP1_Small
- added C? (x2): 100nF, symbol Device:C_Small
- added D? (x2): D_Schottky_Small, symbol Device:D_Schottky_Small
- added MK? (x2): Microphone, symbol Device:Microphone
- added R? (x2): 5.6k, symbol Device:R_Small
- added R? (x2): 2.7k, symbol Device:R_Small
- added R? (x2): 220k, symbol Device:R_Small
- added R? (x4): 100k, symbol Device:R_Small
- added R? (x2): 51k, symbol Device:R_Small
- added R? (x2): 150k, symbol Device:R_Small
- added R? (x2): 12k, symbol Device:R_Small
- added R? (x2): 3k, symbol Device:R_Small
- added R? (x2): 430k, symbol Device:R_Small
- added U? (x3): LM324DT, symbol Device:Opamp_Quad_Generic
- U? (x3): value Opamp_Quad_Generic -> LM324DT
Connections:
- net +5V: now also U?.4 (V+), C?.1, C?.1, R?.1, R?.1, R?.1, R?.1, R?.1, U?.4 (V+)
- net A1: now also C?.2, D?.1 (K), R?.1, R?.2
- net A2: now also C?.2, D?.1 (K), R?.1, R?.2
- net GND: now also U?.11 (V-), C?.2, C?.2, C?.2, D?.2 (A), D?.2 (A), MK?.1 (-), MK?.1 (-), R?.2, R?.2, R?.2, R?.2, R?.2, R?.2, R?.2, U?.11 (V-); no longer U?.10 (+), U?.5 (+)
- net +2V5: now reaches U?.3 (+), U?.3 (+)
- net +2V5: now also U?.10 (+), U?.5 (+), C?.1, R?.1, R?.2, U?.10 (+), U?.5 (+)
- net at U?.6 (-): now also C?.2, R?.2
- net at U?.7: now also C?.1, C?.2, R?.1
- net at U?.8: now also C?.2, R?.1, R?.2
- net at U?.9 (-): now also C?.1, C?.1, R?.1
- new net: C?.2, MK?.2 (+), R?.2 (x2)
- new net: C?.1, C?.1, R?.1, R?.2 (x2)
- new net: C?.2, R?.1, R?.1 (x2)
- new net: C?.1, C?.1, R?.1, U?.6 (-)
- new net: C?.2, R?.1, R?.2, U?.7
- new net: C?.1, R?.2 (x2)
- new net: C?.1, C?.2, R?.1, U?.8
- new net: C?.2, R?.2, U?.9 (-)
Other:
- moved on the sheet: C?, D?, F?, J?, L?, MK?, R?, SW?, U?, U?A, U?B, U?C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
